File: Hardware/Power_Supply.kicad_pcb (KiCad board)
At the start: 2 copper layers, 100 x 50 mm, 67 parts, among them J1 ICSP, J2 Conn_01x01, J3 Conn_01x01, J4 Screw_Terminal_01x02, J6 Conn_01x04, J7 Conn_01x04, SW1 UP, SW2 DW, SW3 V/I, SW4 O_EN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

Commit message: working on 3-d model
Parts:
- removed R11: 10K, Resistor_SMD:R_0805_2012Metric
- removed R3: 665K, Resistor_SMD:R_0805_2012Metric
- removed R4: 130K, Resistor_SMD:R_0805_2012Metric
- removed RL1: ALQ305, relay_ALQ305:ALQ305
- added G***: LOGO, LOGO, F.Cu at (39.0, 29.0)
- added G***: LOGO, LOGO, B.Cu at (39.0, 29.0)
- U3: footprint Package_SO:SOIC-8-1EP_3.9x4.9mm_P1.27mm_EP2.514x3.2mm_ThermalVias -> Package_SO:SOIC-8-1EP_3.9x4.9mm_P1.27mm_EP2.514x3.2mm
- moved C7 15.9 mm to (55.0, 39.0), turned to 180 degrees
- moved U1 0.38 mm to (83.0, 24.6)
Connections:
- R13 pad 1: Net-(R13-Pad1) -> VDC
- U2 pad 30: /~RLY_CNTRL -> /REG_EN
- U3 pad 3: Net-(R3-Pad1) -> /REG_EN
- U5 pad 4: Net-(R13-Pad1) -> VDC
Routing:
- net /REG_EN: track 0.00 -> 41.9 mm, vias 0 -> 4
- net /~RLY_CNTRL: track 39.3 -> 0.00 mm, vias 3 -> 0
- net +5V: track 213.8 -> 201.5 mm, vias 3 -> 5
- net Net-(R3-Pad1): track 7.00 -> 0.00 mm
- net VDC: track 11.4 -> 5.02 mm
- net Net-(R13-Pad1): track 5.02 -> 0.00 mm
- net Net-(C13-Pad2): track 11.0 -> 6.77 mm
- net GND: track 25.7 -> 24.7 mm, vias 83 -> 188
- net Net-(C15-Pad2): track 16.8 -> 16.1 mm
- net /MISO: track 12.5 -> 11.9 mm
- net /SW2: track 25.0 -> 24.4 mm
- net /SW4: track 51.4 -> 50.8 mm
- removed copper zone on F.Cu, net Net-(R13-Pad1)
Other:
- board text added: "+12V | GND"
- board text added: "0.8-12V"
- board text added: "Bench Top PSU V1.0"
- board text added: "GND"
- board text added: "GND | +12V"
- board text removed: "ADSEHGAL"
