File: Hardware V1.0/Power_Supply.kicad_pcb (KiCad board)
At the start: 2 copper layers, 100 x 50 mm, 65 parts, among them J1 ICSP, J2 Conn_01x01, J3 Conn_01x01, J4 Screw_Terminal_01x02, J6 Conn_01x04, J7 Conn_01x04, SW1 UP, SW2 DW, SW3 V/I, SW4 O_EN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

Commit message: added esp32 to schematic
Parts:
- removed J1: ICSP, Custom_Vertical_2x_2.54mm_Pin_Header:PinHeader_2x03_P2.54mm_Vertical
- removed J6, J7: Conn_01x04, Custom_Vertical_1x_2.54mm_Pin_Header:PinHeader_1x04_P2.54mm_Vertical
- added C22: 10μF, Capacitor_SMD:C_0805_2012Metric, F.Cu at (200.8, 65.5)
- added C23: 10μF, Capacitor_SMD:C_0805_2012Metric, F.Cu at (227.6, 35.5)
- added C24: 10μF, Capacitor_SMD:C_0805_2012Metric, F.Cu at (187.5, 72.0)
- added C25: 10μF, Capacitor_SMD:C_0805_2012Metric, F.Cu at (197.8, 59.6)
- added C26: 100nF, Capacitor_SMD:C_0805_2012Metric, F.Cu at (191.9, 72.0)
- added C27: 100nF, Capacitor_SMD:C_0805_2012Metric, F.Cu at (217.1, 41.1)
- added C28: 15nF, Capacitor_SMD:C_0805_2012Metric, F.Cu at (221.6, 39.4)
- added C29: 15nF, Capacitor_SMD:C_0805_2012Metric, F.Cu at (191.9, 69.1)
- added C30: 180pF, Capacitor_SMD:C_0805_2012Metric, F.Cu at (171.7, 83.7)
- added C31: 180pF, Capacitor_SMD:C_0805_2012Metric, F.Cu at (201.2, 53.6)
- added C32: 10pF, Capacitor_SMD:C_0805_2012Metric, F.Cu at (177.0, 80.6)
- added C33: 10pF, Capacitor_SMD:C_0805_2012Metric, F.Cu at (227.6, 29.6)
- added C34: 47µF, Capacitor_SMD:C_0805_2012Metric, F.Cu at (218.4, 47.0)
- added C35: 47µF, Capacitor_SMD:C_0805_2012Metric, F.Cu at (167.3, 84.4)
- added C36: 47µF, Capacitor_SMD:C_0805_2012Metric, F.Cu at (209.2, 50.6)
- added C37: 47µF, Capacitor_SMD:C_0805_2012Metric, F.Cu at (196.3, 69.3)
- added C38: 10uF, Capacitor_SMD:C_Elec_5x5.4, F.Cu at (196.5, 37.7)
- added C39: 100nF, Capacitor_SMD:C_0805_2012Metric, F.Cu at (215.0, 44.0)
- added C40: C_Small, Capacitor_SMD:C_0805_2012Metric, F.Cu at (212.7, 41.1)
- added C41: C_Small, Capacitor_SMD:C_0805_2012Metric, F.Cu at (181.4, 79.5)
- added D4: B320, Diode_SMD:D_SMA, F.Cu at (184.5, 65.2)
- added D5: B320, Diode_SMD:D_SMA, F.Cu at (198.6, 49.9)
- added L2: 3μH, Inductor_SMD:L_Sunlord_MWSA0518_5.4x5.2mm, F.Cu at (217.2, 31.5)
- added L3: 3μH, Inductor_SMD:L_Sunlord_MWSA0518_5.4x5.2mm, F.Cu at (206.8, 38.4)
- added R11: 150K, Resistor_SMD:R_0805_2012Metric, F.Cu at (210.6, 44.0)
- added R21: 18K, Resistor_SMD:R_0805_2012Metric, F.Cu at (232.0, 32.5)
- added R22: 1M, Resistor_SMD:R_0805_2012Metric, F.Cu at (204.8, 50.6)
- added R23: 1M, Resistor_SMD:R_0805_2012Metric, F.Cu at (206.6, 59.5)
- added R24: 75K, Resistor_SMD:R_0805_2012Metric, F.Cu at (182.7, 76.6)
- added R25: 75K, Resistor_SMD:R_0805_2012Metric, F.Cu at (187.1, 75.0)
- added R26: 10K, Resistor_SMD:R_0805_2012Metric, F.Cu at (191.5, 75.0)
- added R27: 3.2K, Resistor_SMD:R_0805_2012Metric, F.Cu at (227.6, 32.5)
- added R28: 38K, Resistor_SMD:R_0805_2012Metric, F.Cu at (210.0, 53.5)
- added R29: 10K, Resistor_SMD:R_0805_2012Metric, F.Cu at (223.2, 35.5)
- added R3: 150K, Resistor_SMD:R_0805_2012Metric, F.Cu at (196.3, 66.4)
- added R30: 0.01R, Resistor_SMD:R_1020_2550Metric, F.Cu at (157.7, 86.0)
- added R31: 500K, Resistor_SMD:R_0805_2012Metric, F.Cu at (176.1, 83.7)
- added R32: 38K, Resistor_SMD:R_0805_2012Metric, F.Cu at (185.8, 80.9)
- added R33: 10K, Resistor_SMD:R_0805_2012Metric, F.Cu at (200.0, 62.5)
- added R4: 18K, Resistor_SMD:R_0805_2012Metric, F.Cu at (223.2, 32.5)
- added U10: INA138, Package_TO_SOT_SMD:SOT-23-5, F.Cu at (162.6, 85.3)
- added U11: LM358, Package_SO:SOIC-8_3.9x4.9mm_P1.27mm, F.Cu at (198.8, 44.4)
- added U12: MCP4023-103ECH, Package_TO_SOT_SMD:SOT-23-6, F.Cu at (190.9, 65.3)
- added U7: TPS45332, Package_SO:SOP-8-1EP_4.57x4.57mm_P1.27mm_EP4.57x4.45mm, F.Cu at (198.7, 31.2)
- added U8: TPS45332, Package_SO:SOP-8-1EP_4.57x4.57mm_P1.27mm_EP4.57x4.45mm, F.Cu at (137.3, 79.3)
- added U9: ESP32-S2-WROVER-I, RF_Module:ESP32-S2-WROVER, F.Cu at (92.3, 37.0)
- D1: value CC -> CC_LED
- D2: value OUT -> OUT_LED
- SW3: value V/I -> V_I_SEL
- moved R15 163.4 mm to (236.4, 29.6)
- moved C16 159.2 mm to (218.0, 50.0), turned to 0 degrees
- moved C20 159.1 mm to (211.0, 56.5), turned to 0 degrees
- moved U5 158.6 mm to (212.9, 37.3), turned to 0 degrees
- moved R18 154.8 mm to (209.6, 47.6)
- moved C7 154.4 mm to (209.2, 31.6), turned to 0 degrees
- moved R19 152.7 mm to (236.4, 32.5), turned to 0 degrees
- moved C3 152.2 mm to (232.0, 35.5)
- moved C18 147.8 mm to (206.6, 56.5), turned to 0 degrees
- moved C13 145.7 mm to (226.0, 41.4), turned to 0 degrees
- moved C6 145.4 mm to (221.6, 42.3), turned to 0 degrees
- moved R14 143.4 mm to (214.4, 53.5), turned to 0 degrees
- moved R12 142.4 mm to (213.6, 50.6)
- moved C21 142.2 mm to (223.2, 29.6), turned to 0 degrees
- moved C5 136.8 mm to (226.0, 38.5), turned to 0 degrees
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Routing:
- net +5V: track 201.5 -> 39.0 mm, vias 5 -> 0
- net /SCL0: track 106.5 -> 0.00 mm, vias 2 -> 0
- net /SDA0: track 104.5 -> 0.00 mm
- net /I_SENSE: track 82.4 -> 0.00 mm, vias 2 -> 0
- net +VSW: track 63.3 -> 0.00 mm
- net /REG_EN: track 41.9 -> 0.00 mm, vias 4 -> 0
- net /SW4: track 50.8 -> 10.3 mm, vias 2 -> 0
- net /V_SENSE: track 37.4 -> 0.00 mm, vias 4 -> 0
- net /POT_U~D: track 27.2 -> 0.00 mm, vias 5 -> 0
- net /SW1: track 36.7 -> 10.1 mm, vias 2 -> 0
- net /~POT_CS: track 26.0 -> 0.00 mm, vias 4 -> 0
- net Net-(C16-Pad2): track 24.5 -> 0.00 mm
- net /RST: track 18.2 -> 0.00 mm, vias 1 -> 0
- net Net-(C15-Pad2): track 16.1 -> 0.00 mm
- net /V_FB: track 15.4 -> 0.00 mm, vias 2 -> 0
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- removed copper zone on F.Cu, net +VSW
- removed copper zone on F.Cu, net Net-(C16-Pad2)
- removed copper zone on F.Cu, net Net-(C6-Pad2)
- removed copper zone on F.Cu, net VDC
Other:
- outline, holes or cut-outs redrawn
