File: Hardware V1.0/Power_Supply.kicad_sch (KiCad schematic)
At the start: 111 parts, among them J1 ICSP, J2 Conn_01x01, J3 Conn_01x01, J4 Screw_Terminal_01x02, J6 Conn_01x04, J7 Conn_01x04, SW1 UP, SW2 DW, SW3 V_I_SEL, SW4 O_EN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

Commit message: added esp32 to schematic
Parts:
- removed U?: ESP32-S2-WROVER-I, RF_Module:ESP32-S2-WROVER, symbol RF_Module:ESP32-S2-WROVER-I
- added D?: 3V3, LED_SMD:LED_0805_2012Metric, symbol Device:LED_Small
- added R?: 330R, Resistor_SMD:R_0805_2012Metric, symbol Device:R_Small_US
- gave numbers to parts that had none: 45
Connections:
- net +3V3: now also R?.2
- net GND: now also D?.1 (K)
- new net: D?.2 (A), R?.1
Other:
- added sheet USB&MCU (USB&MCU.kicad_sch)
- moved on the sheet: C33, C35, C37
