File: V2.0/Hardware/DC_DC_Converter/KiCad_Project_Files/Power_Supply.kicad_sch (KiCad schematic)
At the start: 104 parts, among them J2 Conn_01x01, J3 Conn_01x01, J4 Screw_Terminal_01x02, J5 USB_C_Receptacle_USB2.0, Q1 FDN335N, Q2 FDN335N, Q3 FDN335N, SW1 UP, SW2 DW, SW3 V_I_SEL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

Commit message: esp32 init
Parts:
- added C?: 10µF, Capacitor_SMD:C_0805_2012Metric, symbol Device:C_Small
- added C?: 100nF, Capacitor_SMD:C_0805_2012Metric, symbol Device:C_Small
- added U?: ESP32S2_Wroom, Custom_MCUs:ESP32S2_Wroom, symbol Custom_MCUs:ESP32S2_Wroom
Connections:
- net +3V3: now also C?.2, C?.2, U?.2 (3V3)
- net GND: now also C?.1, C?.1, U?.1 (GND)
Changed lines of the file:
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@@
   (junction (at 97.79 31.115) (diameter 1.016) (color 0 0 0 0))
   (junction (at 97.79 45.085) (diameter 1.016) (color 0 0 0 0))
+  (junction (at 102.87 236.22) (diameter 1.016) (color 0 0 0 0))
   (junction (at 104.14 70.485) (diameter 1.016) (color 0 0 0 0))
   (junction (at 106.045 172.72) (diameter 1.016) (color 0 0 0 0))
   (junction (at 106.045 175.26) (diameter 1.016) (color 0 0 0 0))
+  (junction (at 106.68 236.22) (diameter 1.016) (color 0 0 0 0))
   (junction (at 107.315 26.035) (diameter 1.016) (color 0 0 0 0))
   (junction (at 107.315 33.655) (diameter 1.016) (color 0 0 0 0))
@@
   (junction (at 281.94 78.74) (diameter 1.016) (color 0 0 0 0))
   (junction (at 281.94 82.55) (diameter 1.016) (color 0 0 0 0))
+  (no_connect (at 90.805 105.41))
   (no_connect (at 141.605 102.87))
-  (no_connect (at 45.085 120.65))
-  (no_connect (at 45.085 118.11))
-  (no_connect (at 70.485 110.49))
   (no_connect (at 111.76 61.595))
-  (no_connect (at 69.215 61.595))
-  (no_connect (at 78.105 151.765))
   (no_connect (at 172.085 102.87))
-  (no_connect (at 90.805 105.41))
+  (no_connect (at 70.485 110.49))
+  (no_connect (at 45.085 118.11))
+  (no_connect (at 45.085 120.65))
+  (no_connect (at 78.105 151.765))
+  (no_connect (at 69.215 61.595))
   (wire (pts (xy 12.7 38.1) (xy 15.875 38.1))
     (stroke (width 0) (type solid) (color 0 0 0 0))
@@
     (stroke (width 0) (type solid) (color 0 0 0 0))
   )
+  (wire (pts (xy 99.06 236.22) (xy 102.87 236.22))
+    (stroke (width 0) (type solid) (color 0 0 0 0))
+  )
   (wire (pts (xy 100.965 31.115) (xy 97.79 31.115))
     (stroke (width 0) (type solid) (color 0 0 0 0))
@@
     (stroke (width 0) (type solid) (color 0 0 0 0))
   )
+  (wire (pts (xy 102.87 236.22) (xy 102.87 238.76))
+    (stroke (width 0) (type solid) (color 0 0 0 0))
+  )
+  (wire (pts (xy 102.87 236.22) (xy 106.68 236.22))
+    (stroke (width 0) (type solid) (color 0 0 0 0))
+  )
+  (wire (pts (xy 102.87 247.65) (xy 102.87 243.84))
+    (stroke (width 0) (type solid) (color 0 0 0 0))
+  )
   (wire (pts (xy 104.14 69.215) (xy 104.14 70.485))
     (stroke (width 0) (type solid) (color 0 0 0 0))
@@
     (stroke (width 0) (type solid) (color 0 0 0 0))
   )
+  (wire (pts (xy 106.68 236.22) (xy 106.68 238.76))
+    (stroke (width 0) (type solid) (color 0 0 0 0))
+  )
+  (wire (pts (xy 106.68 236.22) (xy 115.57 236.22))
+    (stroke (width 0) (type solid) (color 0 0 0 0))
+  )
+  (wire (pts (xy 106.68 247.65) (xy 106.68 243.84))
+    (stroke (width 0) (type solid) (color 0 0 0 0))
+  )
   (wire (pts (xy 107.315 26.035) (xy 107.315 27.305))
     (stroke (width 0) (type solid) (color 0 0 0 0))
@@
     (stroke (width 0) (type solid) (color 0 0 0 0))
   )
+  (wire (pts (xy 110.49 233.68) (xy 115.57 233.68))
+    (stroke (width 0) (type solid) (color 0 0 0 0))
+  )
   (wire (pts (xy 111.76 59.055) (xy 116.84 59.055))
     (stroke (width 0) (type solid) (color 0 0 0 0))
@@
     (stroke (width 0) (type solid) (color 0 0 0 0))
   )
-  (wire (pts (xy 149.225 28.575) (xy 151.13 28.575))
+  (wire (pts (xy 149.225 28.575) (xy 153.035 28.575))
     (stroke (width 0) (type solid) (color 0 0 0 0))
   )
@@
     (stroke (width 0) (type solid) (color 0 0 0 0))
   )
-  (wire (pts (xy 151.13 28.575) (xy 153.035 28.575))
-    (stroke (width 0) (type solid) (color 0 0 0 0))
-  )
   (wire (pts (xy 154.94 46.355) (xy 154.94 48.895))
     (stroke (width 0) (type solid) (color 0 0 0 0))
@@
     )
   )
+  (symbol (lib_id "power:+3V3") (at 99.06 236.22 0) (unit 1)
+    (in_bom yes) (on_board yes)
+    (property "Reference" "#PWR?" (id 0) (at 99.06 240.03 0)
+      (effects (font (size 1.27 1.27)) hide)
+    )
+    (property "Value" "+3V3" (id 1) (at 98.425 232.41 0))
+    (property "Footprint" "" (id 2) (at 99.06 236.22 0)
+      (effects (font (size 1.27 1.27)) hide)
+    )
+    (property "Datasheet" "" (id 3) (at 99.06 236.22 0)
+      (effects (font (size 1.27 1.27)) hide)
+    )
+  )
   (symbol (lib_id "power:+5V") (at 123.825 115.57 0) (unit 1)
     (in_bom yes) (on_board yes)
@@
     )
   )
+  (symbol (lib_id "power:GND") (at 102.87 247.65 0) (unit 1)
+    (in_bom yes) (on_board yes)
+    (property "Reference" "#PWR?" (id 0) (at 102.87 254 0)
+      (effects (font (size 1.27 1.27)) hide)
+    )
+    (property "Value" "GND" (id 1) (at 102.87 251.46 0))
+    (property "Footprint" "" (id 2) (at 102.87 247.65 0)
+      (effects (font (size 1.27 1.27)) hide)
+    )
+    (property "Datasheet" "" (id 3) (at 102.87 247.65 0)
+      (effects (font (size 1.27 1.27)) hide)
+    )
+  )
   (symbol (lib_id "power:GND") (at 104.14 70.485 0) (unit 1)
     (in_bom yes) (on_board yes)
@@
     )
   )
+  (symbol (lib_id "power:GND") (at 106.68 247.65 0) (unit 1)
+    (in_bom yes) (on_board yes)
+    (property "Reference" "#PWR?" (id 0) (at 106.68 254 0)
+      (effects (font (size 1.27 1.27)) hide)
+    )
+    (property "Value" "GND" (id 1) (at 106.68 251.46 0))
+    (property "Footprint" "" (id 2) (at 106.68 247.65 0)
+      (effects (font (size 1.27 1.27)) hide)
+    )
+    (property "Datasheet" "" (id 3) (at 106.68 247.65 0)
+      (effects (font (size 1.27 1.27)) hide)
+    )
+  )
   (symbol (lib_id "power:GND") (at 107.315 48.26 0) (unit 1)
     (in_bom yes) (on_board yes)
@@
     )
   )
+  (symbol (lib_id "power:GND") (at 110.49 233.68 270) (unit 1)
+    (in_bom yes) (on_board yes)
+    (property "Reference" "#PWR?" (id 0) (at 104.14 233.68 0)
+      (effects (font (size 1.27 1.27)) hide)
+    )
+    (property "Value" "GND" (id 1) (at 106.68 233.68 0))
+    (property "Footprint" "" (id 2) (at 110.49 233.68 0)
+      (effects (font (size 1.27 1.27)) hide)
+    )
+    (property "Datasheet" "" (id 3) (at 110.49 233.68 0)
+      (effects (font (size 1.27 1.27)) hide)
+    )
+  )
   (symbol (lib_id "power:GND") (at 129.54 92.075 0) (unit 1)
     (in_bom yes) (on_board yes)
@@
     )
   )
+  (symbol (lib_id "Device:C_Small") (at 102.87 241.3 0) (mirror x) (unit 1)
+    (in_bom yes) (on_board yes)
+    (property "Reference" "C?" (id 0) (at 100.33 237.49 0))
+    (property "Value" "10µF" (id 1) (at 99.06 240.03 0))
+    (property "Footprint" "Capacitor_SMD:C_0805_2012Metric" (id 2) (at 102.87 241.3 0)
+      (effects (font (size 1.27 1.27)) hide)
+    )
+    (property "Datasheet" "~" (id 3) (at 102.87 241.3 0)
+      (effects (font (size 1.27 1.27)) hide)
+    )
+  )
+  (symbol (lib_id "Device:C_Small") (at 106.68 241.3 180) (unit 1)
+    (in_bom yes) (on_board yes)
+    (property "Reference" "C?" (id 0) (at 109.22 237.49 0))
+    (property "Value" "100nF" (id 1) (at 110.49 240.03 0))
+    (property "Footprint" "Capacitor_SMD:C_0805_2012Metric" (id 2) (at 106.68 241.3 0)
+      (effects (font (size 1.27 1.27)) hide)
+    )
+    (property "Datasheet" "~" (id 3) (at 106.68 241.3 0)
+      (effects (font (size 1.27 1.27)) hide)
+    )
+  )
   (symbol (lib_id "Device:C_Small") (at 107.315 29.845 180) (unit 1)
     (in_bom yes) (on_board yes)
@@
     )
   )
+  (symbol (lib_id "Custom_MCUs:ESP32S2_Wroom") (at 118.11 260.35 0) (unit 1)
+    (in_bom yes) (on_board yes)
+    (property "Reference" "U?" (id 0) (at 137.16 222.25 0))
+    (property "Value" "ESP32S2_Wroom" (id 1) (at 137.16 224.79 0))
+    (property "Footprint" "Custom_MCUs:ESP32S2_Wroom" (id 2) (at 174.625 298.45 0)
+      (effects (font (size 1.27 1.27)) hide)
+    )
+    (property "Datasheet" "" (id 3) (at 174.625 298.45 0)
+      (effects (font (size 1.27 1.27)) hide)
+    )
+  )
   (symbol_instances
     (path "/cd8bb8c3-f5df-4499-9c79-087b009bf6b4"
@@
       (reference "#PWR0169") (unit 1) (value "+VSW") (footprint "")
     )
+    (path "/30d0f278-d198-4e4e-a9b4-7eacc2fc70b6"
+      (reference "#PWR?") (unit 1) (value "GND") (footprint "")
+    )
+    (path "/337a196e-0e52-48f3-a48e-5928c37ef430"
+      (reference "#PWR?") (unit 1) (value "GND") (footprint "")
+    )
+    (path "/50f931cd-c08a-45c0-bda4-11d29300f346"
+      (reference "#PWR?") (unit 1) (value "GND") (footprint "")
+    )
+    (path "/63e38898-9488-44e9-8473-d93aca332633"
+      (reference "#PWR?") (unit 1) (value "+3V3") (footprint "")
+    )
     (path "/a216915c-7324-469c-8737-2c3edfb6ea67"
       (reference "C1") (unit 1) (value "10nF") (footprint "Capacitor_SMD:C_0805_2012Metric")
@@
       (reference "C35") (unit 1) (value "100nF") (footprint "Capacitor_SMD:C_0805_2012Metric")
     )
+    (path "/9eb64e2a-25c5-4cf0-8990-a88b217a88d5"
+      (reference "C?") (unit 1) (value "10µF") (footprint "Capacitor_SMD:C_0805_2012Metric")
+    )
+    (path "/bb50ae87-4a82-444b-807c-bc03bf96b537"
+      (reference "C?") (unit 1) (value "100nF") (footprint "Capacitor_SMD:C_0805_2012Metric")
+    )
     (path "/b02026a8-7dc6-42d3-9812-c38db0931d18"
       (reference "D1") (unit 1) (value "CL") (footprint "LED_SMD:LED_0805_2012Metric")
@@
       (reference "U11") (unit 3) (value "LM358") (footprint "Package_SO:MSOP-8_3x3mm_P0.65mm")
     )
+    (path "/1b198354-5662-4ef3-9e27-a2efed92848d"
+      (reference "U?") (unit 1) (value "ESP32S2_Wroom") (footprint "Custom_MCUs:ESP32S2_Wroom")
+    )
     (path "/4d0b8609-8a4e-42e5-b830-596bcfcb09bd"
